File: EagleBoards/Chassis/HRT PDB 17-18/HRT PDB 17-18 schem.brd (EAGLE design)
At the start: 135.9 x 105.1 mm, 48 parts, among them J1 TE-TERM-BLOCK, J2 TE-TERM-BLOCK, M1 PLA5D, M2 PLA5D, M3 PLA5D, M4 PLA5D, M5 PLA5D, M6 PLA5D, U1 TI-DCDC-8THBRICK, U2 TI-DCDC-8THBRICK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

Commit message: pdb rev a
Parts:
- added X1, X2, X3, X4: 22-23-2021, con-molex:22-23-2021
- C1, C12, C2, C3: value (none) -> 10u
- C10, C11, C8, C9: value (none) -> .1u
- C5, C6, C7: value (none) -> 330u
- R4, R5: value (none) -> 2k
- R6: value (none) -> 1k
- R7: value (none) -> 332
- R8: value (none) -> 221
- moved D5 18.5 mm to (124.5, 14.0), turned to 180 degrees
- moved R8 16.3 mm to (119.4, 14.0), turned to 0 degrees
- moved D3 14.2 mm to (106.7, 73.7)
- moved R6 14.0 mm to (101.6, 73.7)
- moved R5 11.4 mm to (116.8, 81.3), turned to 90 degrees
- moved D2 7.18 mm to (116.8, 86.4), turned to 270 degrees
- moved C2 6.35 mm to (35.6, 36.8)
- moved C10 5.84 mm to (95.9, 61.5)
- moved D4 4.02 mm to (82.5, 45.7)
- moved R7 4.02 mm to (82.5, 50.8)
- moved R3 2.90 mm to (95.8, 70.9)
- moved C12 2.84 mm to (53.3, 92.7)
- moved C11 2.54 mm to (116.8, 95.2)
- moved C7 2.54 mm to (102.9, 64.8)
- moved C3 2.54 mm to (58.4, 10.2)
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Connections:
- net 12V: now also X2.1
- net 24V: now also X1.1
- net 3.3V: now also X4.1
- net 5V: now also X3.1
- net GND: now also X1.2, X2.2, X3.2, X4.2
Routing:
- net GND: track 0.00 -> 119.5 mm, vias 0 -> 4
- net 5V: track 0.00 -> 31.2 mm
- net 3.3V: track 0.00 -> 28.6 mm
- net N$4: track 0.00 -> 28.2 mm
- net N$6: track 0.00 -> 26.8 mm
- net N$5: track 0.00 -> 24.3 mm
- net 12V: track 0.00 -> 20.5 mm
- net VCC: track 0.00 -> 4.20 mm
- net 24V: track 0.00 -> 3.97 mm
- net N$9: track 0.00 -> 3.25 mm
- net N$8: track 0.00 -> 3.25 mm
- net N$7: track 0.00 -> 3.25 mm
- net N$3: track 0.00 -> 3.25 mm
- net N$2: track 0.00 -> 3.25 mm
- added copper zone on layer 1, net 12V
- added copper zone on layer 1, net 24V
- added copper zone on layer 1, net 3.3V
- added copper zone on layer 1, net 5V
- added copper zone on layer 1, net VCC
