File: EagleBoards/Chassis/HRT PDB 17-18/HRT PDB 17-18 schem.sch (EAGLE design)
At the start: 48 parts, among them J1 TE-TERM-BLOCK, J2 TE-TERM-BLOCK, M1 PLA5D, M2 PLA5D, M3 PLA5D, M4 PLA5D, M5 PLA5D, M6 PLA5D, U1 TI-DCDC-8THBRICK, U2 TI-DCDC-8THBRICK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

Commit message: pdb rev a
Parts:
- added X1, X2, X3, X4: 22-23-2021, con-molex:22-23-2021
- C1, C12, C2, C3: value (none) -> 10u
- C10, C11, C8, C9: value (none) -> .1u
- C5, C6, C7: value (none) -> 330u
- R4, R5: value (none) -> 2k
- R6: value (none) -> 1k
- R7: value (none) -> 332
- R8: value (none) -> 221
Connections:
- net 12V: now also X2-1.S
- net 24V: now also X1-1.S
- net 3.3V: now also X4-1.S
- net 5V: now also X3-1.S
- net GND: now also X1-2.S, X2-2.S, X3-2.S, X4-2.S
