File: Science/Designs/Main Board/Main Board.kicad_pcb (KiCad board)
At the start: 2 copper layers, 68 parts, among them J1 I2C_OUT, J10 AIR_SENS, J11 MOISTURE_SENS, J12 LIMIT3, J13 LIMIT2, J14 LIMIT1, J15 SERVO3, J16 SERVO2, J17 SERVO1, J18 MOTOR1_SIG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

Commit message: Continued working on main PCB
Parts:
- added D12: 7V2_OK, LEDs:LED_D5.0mm, F.Cu at (195.6, 123.2)
- added P1: LS7366R, Housings_SOIC:SOIC-14_3.9x8.7mm_Pitch1.27mm, F.Cu at (220.8, 44.5)
- added P2: LS7366R, Housings_SOIC:SOIC-14_3.9x8.7mm_Pitch1.27mm, F.Cu at (209.4, 44.5)
- added R13: 270Ω, Resistors_SMD:R_1206_HandSoldering, F.Cu at (191.8, 122.5)
- added U1: SN74HC14N, Housings_SOIC:SOIC-14_3.9x8.7mm_Pitch1.27mm, F.Cu at (191.6, 147.3)
- added U2: TLV2544ID, Housings_SOIC:SOIC-16_3.9x9.9mm_Pitch1.27mm, F.Cu at (96.7, 55.2)
- added U5: ACPL-064L-500E, Housings_SOIC:SOIC-8_3.9x4.9mm_Pitch1.27mm, F.Cu at (116.8, 102.9)
- added U6: ACPL-064L-500E, Housings_SOIC:SOIC-8_3.9x4.9mm_Pitch1.27mm, F.Cu at (124.6, 145.4)
