File: Science/Designs/Main Board/Main Board.kicad_pcb (KiCad board)
At the start: 2 copper layers, 76 parts, among them J1 I2C_OUT, J10 AIR_SENS, J11 MOISTURE_SENS, J12 LIMIT3, J13 LIMIT2, J14 LIMIT1, J15 SERVO3, J16 SERVO2, J17 SERVO1, J18 MOTOR1_SIG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

Commit message: Fixed RPi Footprint
Someone (me) got the outline flipped...
Parts:
- added P3: RPI_HEADER, ScienceFootprints:RPi-3B, F.Cu at (223.3, 91.0)
- added P4: PWR_IN, ScienceFootprints:PHOENIX_1792232, F.Cu at (39.2, 52.9)
- added Y1: 20MHz, ScienceFootprints:HC-49USX, F.Cu at (219.8, 34.3)
- added Y2: 20MHz, ScienceFootprints:HC-49USX, F.Cu at (207.1, 34.3)
- moved D1 153.8 mm to (41.9, 97.8)
- moved D12 153.8 mm to (41.9, 118.1)
- moved D3 153.8 mm to (41.9, 108.0)
- moved R1 153.8 mm to (38.1, 97.1)
- moved R13 153.8 mm to (38.1, 117.4)
- moved R2 153.8 mm to (38.1, 86.9)
- moved R3 153.8 mm to (38.1, 107.4)
- moved D2 153.8 mm to (41.7, 87.6)
- moved R40 44.7 mm to (57.1, 107.4), turned to 90 degrees
- moved C19 35.9 mm to (66.0, 105.4), turned to 180 degrees
- moved R41 32.9 mm to (61.0, 107.2), turned to 90 degrees
- moved U7 28.5 mm to (66.0, 100.3)
- moved C18 17.3 mm to (73.7, 105.4)

Commit message: Added RGB LED footprint, working on layout
Parts:
- added D10: LED_RGB, ScienceFootprints:SLV6A-FKB, F.Cu at (85.1, 167.6)
- added D11: LED_RGB, ScienceFootprints:SLV6A-FKB, F.Cu at (100.3, 167.6)
- added D4: LED_RGB, ScienceFootprints:SLV6A-FKB, F.Cu at (47.0, 167.6)
- added D5: LED_RGB, ScienceFootprints:SLV6A-FKB, F.Cu at (62.2, 167.6)
- added D6: LED_RGB, ScienceFootprints:SLV6A-FKB, F.Cu at (77.5, 167.6)
- added D7: LED_RGB, ScienceFootprints:SLV6A-FKB, F.Cu at (92.7, 167.6)
- added D8: LED_RGB, ScienceFootprints:SLV6A-FKB, F.Cu at (54.6, 167.6)
- added D9: LED_RGB, ScienceFootprints:SLV6A-FKB, F.Cu at (69.8, 167.6)
- RP3: moved to B.Cu
- moved P3 209.5 mm to (14.6, 72.7)
- moved D3 179.1 mm to (212.1, 163.8)
- moved R3 179.1 mm to (208.3, 163.3)
- moved C18 176.2 mm to (243.8, 151.1)
- moved C19 176.2 mm to (236.2, 151.1)
- moved D1 176.2 mm to (212.1, 143.5)
- moved D2 176.2 mm to (211.8, 133.3)
- moved P4 176.2 mm to (209.3, 98.6)
- moved R1 176.2 mm to (208.3, 142.8)
- moved R2 176.2 mm to (208.3, 132.6)
- moved R40 176.2 mm to (227.3, 153.1)
- moved U7 176.2 mm to (236.2, 146.1)
- moved R41 176.2 mm to (231.1, 152.9)
- moved D12 173.9 mm to (212.1, 153.7)
- moved R13 173.9 mm to (208.3, 152.9)
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Routing:
- net /RGB_8B: track 0.00 -> 20.0 mm
- net /RGB_4B: track 0.00 -> 19.7 mm
- net /RGB_8G: track 0.00 -> 18.4 mm
- net /RGB_4G: track 0.00 -> 18.3 mm
- net /RGB_8R: track 0.00 -> 17.0 mm
- net /RGB_4R: track 0.00 -> 17.0 mm
- net /RGB_3B: track 0.00 -> 13.7 mm
- net /LED_8B: track 0.00 -> 13.7 mm
- net /LED_4B: track 0.00 -> 13.7 mm
- net /LED_8G: track 0.00 -> 13.4 mm
- net /RGB_7B: track 0.00 -> 12.9 mm
- net /LED_4G: track 0.00 -> 12.7 mm
- net /RGB_3G: track 0.00 -> 12.3 mm
- net /LED_5G: track 0.00 -> 11.7 mm
- net /RGB_7G: track 0.00 -> 11.7 mm
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Other:
- net class Default: clearance 0.2 -> 0.254; trace_width 0.25 -> 0.381; via_dia 0.6 -> 0.508; via_drill 0.4 -> 0.381
- rule trace_clearance: 0.2 -> 0.254

Commit message: Working on PCB
Parts:
- moved J17 48.2 mm to (101.6, 162.6), turned to 90 degrees
- moved U5 48.1 mm to (104.1, 149.2), turned to 90 degrees
- moved R37 42.0 mm to (99.7, 149.3), turned to 90 degrees
- moved J16 37.6 mm to (110.5, 162.6), turned to 90 degrees
- moved C16 36.6 mm to (104.1, 143.5)
- moved R38 29.5 mm to (108.6, 149.2), turned to 90 degrees
- moved J15 29.3 mm to (119.4, 162.6), turned to 90 degrees
- moved R39 21.1 mm to (112.4, 149.2), turned to 90 degrees
- moved C11 17.5 mm to (83.3, 133.1)
- moved C10 17.0 mm to (50.8, 133.3)
- moved RP1 17.0 mm to (50.8, 164.5)
- moved RP2 17.0 mm to (81.3, 164.5)
- moved U3 17.0 mm to (50.8, 139.7)
- moved U4 17.0 mm to (81.3, 139.7)
- moved RP3 17.0 mm to (66.0, 139.1)
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Connections:
- C16 pad 1: +3V3 -> +5V
- C17 pad 1: +3V3 -> +5V

Commit message: Continuing PCB some more
Parts:
- RP1, RP2: moved to B.Cu
- moved C8 150.0 mm to (46.3, 100.3)
- moved U1 150.0 mm to (47.0, 92.5)
- moved R42 143.7 mm to (87.6, 106.7), turned to 90 degrees
- moved P1 139.6 mm to (94.0, 102.9), turned to 180 degrees
- moved D3 137.1 mm to (124.5, 58.4)
- moved C13 136.8 mm to (94.0, 109.2), turned to 180 degrees
- moved R3 136.7 mm to (120.7, 58.4)
- moved D12 136.1 mm to (124.5, 49.5)
- moved R13 135.5 mm to (120.7, 49.5)
- moved Y1 130.7 mm to (108.0, 94.0), turned to 180 degrees
- moved R43 127.5 mm to (87.6, 90.2), turned to 90 degrees
- moved P2 122.8 mm to (94.0, 86.4), turned to 180 degrees
- moved C5 121.3 mm to (102.9, 100.3), turned to 270 degrees
- moved C12 120.7 mm to (94.0, 92.7), turned to 180 degrees
- moved R11 120.2 mm to (106.7, 100.3), turned to 270 degrees
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Routing:
- net /LED_8B: track 13.7 -> 0.00 mm
- net /LED_4B: track 13.7 -> 0.00 mm
- net /LED_8G: track 13.4 -> 0.00 mm
- net /LED_4G: track 12.7 -> 0.00 mm
- net Net-(C7-Pad1): track 0.00 -> 12.2 mm
- net Net-(C5-Pad1): track 0.00 -> 12.2 mm
- net /LED_5G: track 11.7 -> 0.00 mm
- net /LED_5B: track 11.5 -> 0.00 mm
- net /LED_1G: track 11.2 -> 0.00 mm
- net /LED_1B: track 10.9 -> 0.00 mm
- net /LED_7B: track 9.71 -> 0.00 mm
- net /LED_7G: track 9.14 -> 0.00 mm
- net /LED_3B: track 9.08 -> 0.00 mm
- net /LED_3G: track 8.51 -> 0.00 mm
- net Net-(C6-Pad1): track 0.00 -> 8.20 mm
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Other:
- board outline added: 114.3 x 101.6 mm
- net class Default: trace_width 0.381 -> 0.508

Commit message: Continued continuing on main board
Parts:
- added HS1: HEATSINK, ScienceFootprints:AAVID_531202B02500G, F.Cu at (125.1, 110.5)
- moved C17 59.2 mm to (68.3, 91.8), turned to 90 degrees
- moved U6 57.0 mm to (74.0, 91.8), turned to 180 degrees
- moved R39 50.9 mm to (74.0, 96.2), turned to 180 degrees
- moved R38 45.6 mm to (74.0, 100.0), turned to 180 degrees
- moved C16 42.8 mm to (68.3, 104.5), turned to 90 degrees
- moved U5 39.6 mm to (74.0, 104.5), turned to 180 degrees
- moved R37 33.6 mm to (74.1, 108.9), turned to 180 degrees
- moved RP1 5.08 mm to (54.6, 132.1)
- moved RP2 5.08 mm to (85.1, 132.1)
- moved C10 1.91 mm to (54.6, 117.5)
Routing:
- net /LED_1R: track 0.00 -> 36.8 mm, vias 0 -> 1
- net /LED_7R: track 0.00 -> 34.0 mm, vias 0 -> 1
- net /LED_2R: track 0.00 -> 33.3 mm, vias 0 -> 1
- net /LED_8R: track 0.00 -> 31.3 mm, vias 0 -> 1
- net /RGB_1R: track 0.00 -> 27.0 mm
- net /LED_3R: track 0.00 -> 26.9 mm, vias 0 -> 1
- net /RGB_1G: track 0.00 -> 23.5 mm
- net /LED_4R: track 0.00 -> 23.3 mm, vias 0 -> 1
- net /RGB_1B: track 0.00 -> 20.6 mm
- net /LED_6R: track 0.00 -> 19.3 mm, vias 0 -> 1
- net /RGB_2R: track 0.00 -> 14.5 mm
- net /LED_5R: track 0.00 -> 13.9 mm, vias 0 -> 1
- net /LED_8B: track 0.00 -> 13.8 mm, vias 0 -> 1
- net /LED_4B: track 0.00 -> 13.8 mm, vias 0 -> 1
- net /LED_4G: track 0.00 -> 13.2 mm, vias 0 -> 1
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
Commit message: Finishing up for tonight.
Parts:
- moved P7 5.08 mm to (47.0, 63.5)
- moved P9 5.08 mm to (47.0, 68.6)
Connections:
- P6 pad 5: /PI_SDA -> /PI_SCL
Routing:
- net +3V3: track 0.00 -> 81.0 mm
- net /PI_SDA: track 0.00 -> 35.1 mm
- net /PI_SCL: track 0.00 -> 32.3 mm
- net /RGB_5R: track 0.00 -> 27.2 mm
- net /RGB_5G: track 0.00 -> 23.5 mm
- net /RGB_5B: track 0.00 -> 20.2 mm
- net /RGB_6R: track 0.00 -> 14.5 mm
- net +5V: track 0.00 -> 8.89 mm
- net Net-(J10-Pad2): track 0.00 -> 8.42 mm
- net Net-(J2-Pad2): track 0.00 -> 8.42 mm
- net Net-(J11-Pad2): track 0.00 -> 8.42 mm
- net /LED_7R: track 34.0 -> 40.4 mm
- net /MOIST_SENS_OUT: track 0.00 -> 3.81 mm
- net /AQ_SENS_OUT: track 0.00 -> 3.81 mm
- net /ANE_SENS_OUT: track 0.00 -> 3.81 mm
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
Commit message: More layout
Parts:
- moved C10 10.8 mm to (61.6, 125.7), turned to 270 degrees
- moved C11 1.02 mm to (87.6, 120.0)
Routing:
- net /PI_MISO: track 0.00 -> 100.8 mm
- net /PI_SCK: track 0.00 -> 98.3 mm
- net /PI_SDA: track 35.1 -> 70.8 mm, vias 0 -> 2
- net /PI_SCL: track 32.3 -> 66.4 mm, vias 0 -> 2
- net /PI_MOSI: track 0.00 -> 26.7 mm, vias 0 -> 1
- net +3V3: track 81.0 -> 98.0 mm
- net /ANE_SENS_OUT: track 3.81 -> 20.0 mm, vias 0 -> 2
- net /AQ_SENS_OUT: track 3.81 -> 16.2 mm, vias 0 -> 2
- net /MOIST_SENS_OUT: track 3.81 -> 14.9 mm, vias 0 -> 2
- net Net-(D2-Pad1): track 0.00 -> 5.38 mm
- net Net-(D1-Pad1): track 0.00 -> 5.38 mm
- net Net-(D3-Pad1): track 0.00 -> 5.38 mm
- net Net-(D12-Pad1): track 0.00 -> 5.38 mm
Other:
- rule trace_min: 0.2 -> 0.2032
- rule via_min_drill: 0.3 -> 0.3048
- rule via_min_size: 0.4 -> 0.381

Commit message: Even more layout
Parts:
- added REF**: MountingHole_3.2mm_M3_Pad_Via, Mounting_Holes:MountingHole_3.2mm_M3_Pad_Via, F.Cu at (139.7, 141.0)
- added REF**: MountingHole_3.2mm_M3_Pad_Via, Mounting_Holes:MountingHole_3.2mm_M3_Pad_Via, F.Cu at (139.7, 49.5)
- added REF**: MountingHole_3.2mm_M3_Pad_Via, Mounting_Holes:MountingHole_3.2mm_M3_Pad_Via, F.Cu at (22.9, 49.5)
- added REF**: MountingHole_3.2mm_M3_Pad_Via, Mounting_Holes:MountingHole_3.2mm_M3_Pad_Via, F.Cu at (22.9, 141.0)
- moved J12 68.7 mm to (111.8, 50.8), turned to 90 degrees
- moved J13 56.9 mm to (120.7, 50.8), turned to 90 degrees
- moved R1 53.1 mm to (180.3, 77.5)
- moved R13 53.1 mm to (170.2, 68.6)
- moved R2 53.1 mm to (180.3, 68.6)
- moved R3 53.1 mm to (170.2, 77.5)
- moved D12 47.8 mm to (133.3, 96.5)
- moved D2 47.3 mm to (139.7, 96.5)
- moved J14 45.4 mm to (129.5, 50.8), turned to 90 degrees
- moved D3 45.3 mm to (133.3, 102.9)
- moved D1 44.7 mm to (139.7, 102.9)
- moved J1 27.9 mm to (137.2, 87.6), turned to 0 degrees
- moved J15 8.13 mm to (137.2, 114.3)
- moved J16 8.13 mm to (137.2, 123.2)
- moved J17 8.13 mm to (137.2, 132.1), turned to 0 degrees
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Routing:
- net +3V3: track 98.0 -> 176.4 mm
Other:
- board size 114.3 x 101.6 mm -> 127 x 101.6 mm
- board text added: "1"
- board text added: "2"
- board text added: "3"
- board text added: "ENCODER"
- board text added: "LIMIT SW"
