File: Science/Designs/Main Board/_saved_Main Board.sch (KiCad schematic (older format))
At the start: 89 parts, among them J1 I2C_OUT, J10 AIR_SENS, J11 MOISTURE_SENS, J12 LIMIT3, J13 LIMIT2, J14 LIMIT1, J15 SERVO3, J16 SERVO2, J17 SERVO1, J18 MOTOR1_SIG, J19 MOTOR2_SIG, J2 ANE_SENS, J20 MOTOR3_SIG, J4 ENCODER2, J5 ENCODER1, J7 ATMO_SENS, P1 LS7366R, P2 LS7366R, P3 RPI_HEADER, P4 PWR_IN, P5 UV_SENS, P6 DIST_SENS, P7 I2C_TEST, P8 THERMO_SENS, P9 SPI_TEST, U1 SN74HC14N, U2 TLV2544ID, U3 PCA9685, U4 PCA9685, U5 ACPL-064L-500E, U6 ACPL-064L-500E, U7 LM317T, Y1 20MHz, Y2 20MHz

Commit message: Added RGB LED footprint, working on layout
Parts:
- D10, D11, D4, D5, D6, D7, D8, D9: footprint (none) -> ScienceFootprints:SLV6A-FKB
- Y1, Y2: footprint (none) -> ScienceFootprints:HC-49USX
Changed lines of the file:
@@
 F 0 "Y1" H 8900 4600 50  0000 C CNN
 F 1 "20MHz" H 8900 4300 35  0000 C CNN
-F 2 "" H 8900 4450 50  0001 C CNN
+F 2 "ScienceFootprints:HC-49USX" H 8900 4450 50  0001 C CNN
 F 3 "" H 8900 4450 50  0001 C CNN
 	1    8900 4450
@@
 F 0 "Y2" H 8900 5650 50  0000 C CNN
 F 1 "20MHz" H 8900 5350 35  0000 C CNN
-F 2 "" H 8900 5500 50  0001 C CNN
+F 2 "ScienceFootprints:HC-49USX" H 8900 5500 50  0001 C CNN
 F 3 "" H 8900 5500 50  0001 C CNN
 	1    8900 5500
@@
 F 0 "D4" H 7350 1475 50  0000 C CNN
 F 1 "LED_RGB" H 7350 1400 50  0000 C CNN
-F 2 "" H 7350 1000 50  0001 C CNN
+F 2 "ScienceFootprints:SLV6A-FKB" H 7350 1000 50  0001 C CNN
 F 3 "" H 7350 1000 50  0000 C CNN
 	1    7350 1050
@@
 F 0 "D5" H 7350 2275 50  0000 C CNN
 F 1 "LED_RGB" H 7350 2200 50  0000 C CNN
-F 2 "" H 7350 1800 50  0001 C CNN
+F 2 "ScienceFootprints:SLV6A-FKB" H 7350 1800 50  0001 C CNN
 F 3 "" H 7350 1800 50  0000 C CNN
 	1    7350 1850
@@
 F 0 "D6" H 7350 3075 50  0000 C CNN
 F 1 "LED_RGB" H 7350 3000 50  0000 C CNN
-F 2 "" H 7350 2600 50  0001 C CNN
+F 2 "ScienceFootprints:SLV6A-FKB" H 7350 2600 50  0001 C CNN
 F 3 "" H 7350 2600 50  0000 C CNN
 	1    7350 2650
@@
 F 0 "D7" H 7350 3875 50  0000 C CNN
 F 1 "LED_RGB" H 7350 3800 50  0000 C CNN
-F 2 "" H 7350 3400 50  0001 C CNN
+F 2 "ScienceFootprints:SLV6A-FKB" H 7350 3400 50  0001 C CNN
 F 3 "" H 7350 3400 50  0000 C CNN
 	1    7350 3450
@@
 F 0 "D8" H 8300 1475 50  0000 C CNN
 F 1 "LED_RGB" H 8300 1400 50  0000 C CNN
-F 2 "" H 8300 1000 50  0001 C CNN
+F 2 "ScienceFootprints:SLV6A-FKB" H 8300 1000 50  0001 C CNN
 F 3 "" H 8300 1000 50  0000 C CNN
 	1    8300 1050
@@
 F 0 "D9" H 8300 2275 50  0000 C CNN
 F 1 "LED_RGB" H 8300 2200 50  0000 C CNN
-F 2 "" H 8300 1800 50  0001 C CNN
+F 2 "ScienceFootprints:SLV6A-FKB" H 8300 1800 50  0001 C CNN
 F 3 "" H 8300 1800 50  0000 C CNN
 	1    8300 1850
@@
 F 0 "D10" H 8300 3075 50  0000 C CNN
 F 1 "LED_RGB" H 8300 3000 50  0000 C CNN
-F 2 "" H 8300 2600 50  0001 C CNN
+F 2 "ScienceFootprints:SLV6A-FKB" H 8300 2600 50  0001 C CNN
 F 3 "" H 8300 2600 50  0000 C CNN
 	1    8300 2650
@@
 F 0 "D11" H 8300 3875 50  0000 C CNN
 F 1 "LED_RGB" H 8300 3800 50  0000 C CNN
-F 2 "" H 8300 3400 50  0001 C CNN
+F 2 "ScienceFootprints:SLV6A-FKB" H 8300 3400 50  0001 C CNN
 F 3 "" H 8300 3400 50  0000 C CNN
 	1    8300 3450
