File: Science/Designs/Power Board/_saved_Power Board.sch (KiCad schematic (older format))
At the start: 25 parts

Commit message: Began Power Board layout
Parts:
- C1, C2, C3: renamed from C?; footprint (none) -> Capacitors_SMD:C_1206_HandSoldering
- D1, D2, D3, D4: renamed from D?; footprint (none) -> LEDs:LED_D5.0mm; symbol LED -> LED-RESCUE-Power_Board
- P1, P5: renamed from P?; footprint (none) -> ScienceFootprints:PHOENIX_1792229
- P2: renamed from P?; footprint (none) -> ScienceFootprints:PHOENIX_1792245
- P3, P6, P7: renamed from P?; footprint (none) -> ScienceFootprints:PHOENIX_1792232
- P4: renamed from P?; footprint (none) -> ScienceFootprints:MOLEX_22-23-2041
- R1, R2, R3, R4, R5, R6, R7, R8: renamed from R?; footprint (none) -> Resistors_SMD:R_1206_HandSoldering
- U1, U2, U3: renamed from U?; footprint (none) -> Housings_SOIC:SO-8_5.3x6.2mm_Pitch1.27mm

Commit message: Updated footprint library
Parts:
- R1, R3: footprint Resistors_SMD:R_1206_HandSoldering -> ScienceFootprints:2526W
- R4: footprint Resistors_SMD:R_1206_HandSoldering -> ScienceFootprints:2827W
- R5: footprint Resistors_SMD:R_1206_HandSoldering -> Resistors_THT:R_Axial_Power_L25.0mm_W6.4mm_P30.48mm
Changed lines of the file:
@@
 F 0 "R3" V 2530 2100 50  0000 C CNN
 F 1 "2mΩ" V 2450 2100 50  0000 C CNN
-F 2 "Resistors_SMD:R_1206_HandSoldering" V 2380 2100 50  0001 C CNN
+F 2 "ScienceFootprints:2526W" V 2380 2100 50  0001 C CNN
 F 3 "" H 2450 2100 50  0000 C CNN
 	1    2450 2100
@@
 F 0 "R4" V 2530 2750 50  0000 C CNN
 F 1 "10mΩ" V 2450 2750 50  0000 C CNN
-F 2 "Resistors_SMD:R_1206_HandSoldering" V 2380 2750 50  0001 C CNN
+F 2 "ScienceFootprints:2827W" V 2380 2750 50  0001 C CNN
 F 3 "" H 2450 2750 50  0000 C CNN
 	1    2450 2750
@@
 F 0 "R5" V 3080 3850 50  0000 C CNN
 F 1 "150mΩ" V 3000 3850 39  0000 C CNN
-F 2 "Resistors_SMD:R_1206_HandSoldering" V 2930 3850 50  0001 C CNN
+F 2 "Resistors_THT:R_Axial_Power_L25.0mm_W6.4mm_P30.48mm" V 2930 3850 50  0001 C CNN
 F 3 "" H 3000 3850 50  0000 C CNN
 	1    3000 3850
@@
 F 0 "R1" V 2330 2100 50  0000 C CNN
 F 1 "2mΩ" V 2250 2100 50  0000 C CNN
-F 2 "Resistors_SMD:R_1206_HandSoldering" V 2180 2100 50  0001 C CNN
+F 2 "ScienceFootprints:2526W" V 2180 2100 50  0001 C CNN
 F 3 "" H 2250 2100 50  0000 C CNN
 	1    2250 2100
