File: Science/Designs/Power Board/_saved_Power Board.sch (KiCad schematic (older format))
At the start: 25 parts, among them P1 PWR_IN, P2 MOTOR_PWR_OUT, P3 MAIN_PWR_OUT, P4 I2C, P5 MOTOR_SW, P6 REG_12V, P7 REG_5V, U1 INA226, U2 INA226

Commit message: Replaced current sensor with INA226
Parts:
- U3: renamed from U?; footprint (none) -> Housings_SSOP:MSOP-10_3x3mm_Pitch0.5mm
Changed lines of the file:
@@
 	3700 2750 3700 2700
 $Comp
-L INA226 U?
+L INA226 U3
 U 1 1 5A65DF2C
 P 3700 4050
-F 0 "U?" H 3900 3700 40  0000 C CNN
+F 0 "U3" H 3900 3700 40  0000 C CNN
 F 1 "INA226" H 3700 4400 40  0000 C CNN
-F 2 "" H 3700 4000 40  0001 C CNN
+F 2 "Housings_SSOP:MSOP-10_3x3mm_Pitch0.5mm" H 3700 4000 40  0001 C CNN
 F 3 "" H 3700 4000 40  0001 C CNN
 	1    3700 4050
